File: amiga_floppy.kicad_pcb (KiCad board)
At the start: 2 copper layers, 52 x 68.3 mm, 6 parts

Commit message: added holes
Parts:
- added H0: , MountingHole:MountingHole_2.1mm, F.Cu at (136.2, 138.9)
- added H1: , MountingHole:MountingHole_2.1mm, F.Cu at (189.3, 138.9)
- added H2: , MountingHole:MountingHole_2.1mm, F.Cu at (189.3, 68.2)
- added H3: , MountingHole:MountingHole_2.1mm, F.Cu at (136.2, 68.2)
Routing:
- net (no net): track 823.6 -> 827.8 mm
Other:
- board size 52 x 68.3 mm -> 59.5 x 77.1 mm
